Commit message: sim2sim, sdk2

File: legged_robot_description/g1_description/urdf/g1_29dof_lock_waist_rev_1_0.ros2_control.xacro (robot description, xacro)
@@ -1,9 +1,17 @@
 <?xml version="1.0"?>
 <robot xmlns:xacro="http://www.ros.org/wiki/xacro">
-  <xacro:macro name="g1_29dof_lock_waist_rev_1_0_ros2_control" params="prefix">
+  <xacro:macro name="g1_29dof_lock_waist_rev_1_0_ros2_control" params="prefix enable_sim:=false">
     <ros2_control name="g1_29dof_lock_waist_rev_1_0_ros2_control" type="system">
-      <hardware>
-        <plugin>legged_ros2_control/MujocoSystemInterface</plugin>
-      </hardware>
+      <xacro:if value="${enable_sim}">
+        <hardware>
+          <plugin>legged_ros2_control/MujocoSystemInterface</plugin>
+        </hardware>
+      </xacro:if>
+      <xacro:unless value="${enable_sim}">
+        <hardware>
+          <plugin>legged_ros2_control/G1SystemInterface</plugin>
+          <param name="network_interface">lo</param>
+        </hardware>
+      </xacro:unless>
       <joint name="${prefix}left_hip_pitch_joint">
         <command_interface name="position">
@@ -519,28 +527,44 @@
         <state_interface name="effort" />
       </joint>
-      <sensor name="imu-torso">
-        <state_interface name="orientation.x"/>
-        <state_interface name="orientation.y"/>
-        <state_interface name="orientation.z"/>
-        <state_interface name="orientation.w"/>
-        <state_interface name="angular_velocity.x"/>
-        <state_interface name="angular_velocity.y"/>
-        <state_interface name="angular_velocity.z"/>
-        <state_interface name="linear_acceleration.x"/>
-        <state_interface name="linear_acceleration.y"/>
-        <state_interface name="linear_acceleration.z"/>
-      </sensor>
-      <sensor name="imu-pelvis">
-        <state_interface name="orientation.x"/>
-        <state_interface name="orientation.y"/>
-        <state_interface name="orientation.z"/>
-        <state_interface name="orientation.w"/>
-        <state_interface name="angular_velocity.x"/>
-        <state_interface name="angular_velocity.y"/>
-        <state_interface name="angular_velocity.z"/>
-        <state_interface name="linear_acceleration.x"/>
-        <state_interface name="linear_acceleration.y"/>
-        <state_interface name="linear_acceleration.z"/>
-      </sensor>
+      <xacro:if value="${enable_sim}">
+        <sensor name="imu-torso">
+          <state_interface name="orientation.x"/>
+          <state_interface name="orientation.y"/>
+          <state_interface name="orientation.z"/>
+          <state_interface name="orientation.w"/>
+          <state_interface name="angular_velocity.x"/>
+          <state_interface name="angular_velocity.y"/>
+          <state_interface name="angular_velocity.z"/>
+          <state_interface name="linear_acceleration.x"/>
+          <state_interface name="linear_acceleration.y"/>
+          <state_interface name="linear_acceleration.z"/>
+        </sensor>
+        <sensor name="imu-pelvis">
+          <state_interface name="orientation.x"/>
+          <state_interface name="orientation.y"/>
+          <state_interface name="orientation.z"/>
+          <state_interface name="orientation.w"/>
+          <state_interface name="angular_velocity.x"/>
+          <state_interface name="angular_velocity.y"/>
+          <state_interface name="angular_velocity.z"/>
+          <state_interface name="linear_acceleration.x"/>
+          <state_interface name="linear_acceleration.y"/>
+          <state_interface name="linear_acceleration.z"/>
+        </sensor>
+      </xacro:if>
+      <xacro:unless value="${enable_sim}">
+        <sensor name="imu-pelvis">
+          <state_interface name="orientation.x"/>
+          <state_interface name="orientation.y"/>
+          <state_interface name="orientation.z"/>
+          <state_interface name="orientation.w"/>
+          <state_interface name="angular_velocity.x"/>
+          <state_interface name="angular_velocity.y"/>
+          <state_interface name="angular_velocity.z"/>
+          <state_interface name="linear_acceleration.x"/>
+          <state_interface name="linear_acceleration.y"/>
+          <state_interface name="linear_acceleration.z"/>
+        </sensor>
+      </xacro:unless>
     </ros2_control>
   </xacro:macro>

Commit message: support go2

File: legged_robot_description/g1_description/urdf/g1_29dof_lock_waist_rev_1_0.ros2_control.xacro (robot description, xacro)
@@ -1,5 +1,5 @@
 <?xml version="1.0"?>
 <robot xmlns:xacro="http://www.ros.org/wiki/xacro">
-  <xacro:macro name="g1_29dof_lock_waist_rev_1_0_ros2_control" params="prefix enable_sim:=false">
+  <xacro:macro name="g1_29dof_lock_waist_rev_1_0_ros2_control" params="prefix enable_sim:=false network_interface:=lo">
     <ros2_control name="g1_29dof_lock_waist_rev_1_0_ros2_control" type="system" is_async="true">
       <xacro:if value="${enable_sim}">
@@ -11,5 +11,5 @@
         <hardware>
           <plugin>legged_ros2_control/G1SystemInterface</plugin>
-          <param name="network_interface">lo</param>
+          <param name="network_interface">${network_interface}</param>
         </hardware>
       </xacro:unless>

File: legged_robot_description/g1_description/urdf/g1_29dof_lock_waist_rev_1_0.urdf.xacro (robot description, xacro)
@@ -3,7 +3,11 @@
   <xacro:arg name="prefix" default="" />
   <xacro:arg name="enable_sim" default="true" />
+  <xacro:arg name="network_interface" default="lo" />
   <xacro:include filename="$(find g1_description)/urdf/g1_29dof_lock_waist_rev_1_0_macro.urdf.xacro" />
   <xacro:include filename="$(find g1_description)/urdf/g1_29dof_lock_waist_rev_1_0.ros2_control.xacro" />
   <xacro:g1_29dof_lock_waist_rev_1_0 prefix="$(arg prefix)" />
-  <xacro:g1_29dof_lock_waist_rev_1_0_ros2_control prefix="$(arg prefix)" enable_sim="$(arg enable_sim)"/>
+  <xacro:g1_29dof_lock_waist_rev_1_0_ros2_control
+    prefix="$(arg prefix)"
+    enable_sim="$(arg enable_sim)"
+    network_interface="$(arg network_interface)"/>
 </robot>

File: legged_robot_description/go2_description/xacro/robot.xacro (robot description, xacro)
@@ -2,4 +2,7 @@
 <robot name="go2" xmlns:xacro="http://www.ros.org/wiki/xacro">
     <xacro:arg name="DEBUG" default="false"/>
+    <xacro:arg name="prefix" default="" />
+    <xacro:arg name="enable_sim" default="true" />
+    <xacro:arg name="network_interface" default="lo" />
     <xacro:include filename="$(find go2_description)/xacro/const.xacro"/>
     <xacro:include filename="$(find go2_description)/xacro/materials.xacro"/>
@@ -119,4 +122,7 @@
     <xacro:leg name="RR" mirror="-1" mirror_dae="False"  front_hind="-1" front_hind_dae="False" />
     <xacro:leg name="RL" mirror="1"  mirror_dae="True"   front_hind="-1" front_hind_dae="False" />
-    <xacro:go2_ros2_control prefix=""/>
+    <xacro:go2_ros2_control
+        prefix="$(arg prefix)"
+        enable_sim="$(arg enable_sim)"
+        network_interface="$(arg network_interface)"/>
 </robot>

File: legged_robot_description/go2_description/xacro/ros2_control.xacro (robot description, xacro)
@@ -1,9 +1,17 @@
 <?xml version="1.0"?>
 <robot xmlns:xacro="http://www.ros.org/wiki/xacro">
-  <xacro:macro name="go2_ros2_control" params="prefix">
+  <xacro:macro name="go2_ros2_control" params="prefix enable_sim:=false network_interface:=lo">
     <ros2_control name="go2_ros2_control" type="system">
-      <hardware>
-        <plugin>legged_ros2_control/MujocoSystemInterface</plugin>
-      </hardware>
+      <xacro:if value="${enable_sim}">
+        <hardware>
+          <plugin>legged_ros2_control/MujocoSystemInterface</plugin>
+        </hardware>
+      </xacro:if>
+      <xacro:unless value="${enable_sim}">
+        <hardware>
+          <plugin>legged_ros2_control/Go2SystemInterface</plugin>
+          <param name="network_interface">${network_interface}</param>
+        </hardware>
+      </xacro:unless>
       <joint name="${prefix}FL_hip_joint">
         <command_interface name="position">
