Commit message: update G1 description

File: legged_robot_description/g1_description/urdf/g1_29dof_rev_1_0.urdf (robot description, URDF)
Before this commit: robot g1_29dof_lock_waist_rev_1_0, 39 links, 38 joints
Links:
- link head_link: geometry collision mesh filename=meshes/head_link.STL; visual mesh filename=meshes/head_link.STL
- link left_ankle_pitch_link: geometry collision mesh filename=meshes/left_ankle_pitch_link.STL; visual mesh filename=meshes/left_ankle_pitch_link.STL
- link left_ankle_roll_link: geometry collision sphere radius=0.005; collision sphere radius=0.005
- link left_elbow_link: geometry collision mesh filename=meshes/left_elbow_link.STL; visual mesh filename=meshes/left_elbow_link.STL
- link left_hip_pitch_link: geometry collision mesh filename=meshes/left_hip_pitch_link.STL; visual mesh filename=meshes/left_hip_pitch_link.STL
- link left_hip_roll_link: geometry collision mesh filename=meshes/left_hip_roll_link.STL; visual mesh filename=meshes/left_hip_roll_link.STL
- link left_hip_yaw_link: geometry collision mesh filename=meshes/left_hip_yaw_link.STL; visual mesh filename=meshes/left_hip_yaw_link.STL
- link left_knee_link: geometry collision mesh filename=meshes/left_knee_link.STL; visual mesh filename=meshes/left_knee_link.STL
- link left_rubber_hand: geometry visual mesh filename=meshes/left_rubber_hand.STL
- link left_shoulder_pitch_link: geometry collision cylinder length=0.05 radius=0.03; visual mesh filename=meshes/left_shoulder_pitch_link.STL
- link left_shoulder_roll_link: geometry collision cylinder length=0.03 radius=0.03; visual mesh filename=meshes/left_shoulder_roll_link.STL
- link left_shoulder_yaw_link: geometry collision mesh filename=meshes/left_shoulder_yaw_link.STL; visual mesh filename=meshes/left_shoulder_yaw_link.STL
- link left_wrist_pitch_link: geometry collision mesh filename=meshes/left_wrist_pitch_link.STL; visual mesh filename=meshes/left_wrist_pitch_link.STL
- link left_wrist_roll_link: geometry collision mesh filename=meshes/left_wrist_roll_link.STL; visual mesh filename=meshes/left_wrist_roll_link.STL
- link left_wrist_yaw_link: geometry collision mesh filename=meshes/left_wrist_yaw_link.STL; visual mesh filename=meshes/left_wrist_yaw_link.STL
- link logo_link: geometry collision mesh filename=meshes/logo_link.STL; visual mesh filename=meshes/logo_link.STL
- link pelvis: geometry visual mesh filename=meshes/pelvis.STL
- link pelvis_contour_link: geometry collision mesh filename=meshes/pelvis_contour_link.STL; visual mesh filename=meshes/pelvis_contour_link.STL
- link right_ankle_pitch_link: geometry collision mesh filename=meshes/right_ankle_pitch_link.STL; visual mesh filename=meshes/right_ankle_pitch_link.STL
- link right_ankle_roll_link: geometry collision sphere radius=0.005; collision sphere radius=0.005
- link right_elbow_link: geometry collision mesh filename=meshes/right_elbow_link.STL; visual mesh filename=meshes/right_elbow_link.STL
- link right_hip_pitch_link: geometry collision mesh filename=meshes/right_hip_pitch_link.STL; visual mesh filename=meshes/right_hip_pitch_link.STL
- link right_hip_roll_link: geometry collision mesh filename=meshes/right_hip_roll_link.STL; visual mesh filename=meshes/right_hip_roll_link.STL
- link right_hip_yaw_link: geometry collision mesh filename=meshes/right_hip_yaw_link.STL; visual mesh filename=meshes/right_hip_yaw_link.STL
- link right_knee_link: geometry collision mesh filename=meshes/right_knee_link.STL; visual mesh filename=meshes/right_knee_link.STL
- link right_rubber_hand: geometry visual mesh filename=meshes/right_rubber_hand.STL
- link right_shoulder_pitch_link: geometry collision cylinder length=0.05 radius=0.03; visual mesh filename=meshes/right_shoulder_pitch_link.STL
- link right_shoulder_roll_link: geometry collision cylinder length=0.03 radius=0.03; visual mesh filename=meshes/right_shoulder_roll_link.STL
- link right_shoulder_yaw_link: geometry collision mesh filename=meshes/right_shoulder_yaw_link.STL; visual mesh filename=meshes/right_shoulder_yaw_link.STL
- link right_wrist_pitch_link: geometry collision mesh filename=meshes/right_wrist_pitch_link.STL; visual mesh filename=meshes/right_wrist_pitch_link.STL
- link right_wrist_roll_link: geometry collision mesh filename=meshes/right_wrist_roll_link.STL; visual mesh filename=meshes/right_wrist_roll_link.STL
- link right_wrist_yaw_link: geometry collision mesh filename=meshes/right_wrist_yaw_link.STL; visual mesh filename=meshes/right_wrist_yaw_link.STL
- link torso_link: geometry collision mesh filename=meshes/torso_link_rev_1_0.STL; visual mesh filename=meshes/torso_link_rev_1_0.STL
- link waist_roll_link: geometry visual mesh filename=meshes/waist_roll_link_rev_1_0.STL
- link waist_yaw_link: geometry visual mesh filename=meshes/waist_yaw_link_rev_1_0.STL
Joints:
- joint waist_pitch_joint: type fixed -> revolute
- joint waist_roll_joint: type fixed -> revolute

File: legged_robot_description/g1_description/urdf/g1_29dof_rev_1_0_macro.urdf.xacro (robot description, xacro)
@@ -1,4 +1,4 @@
 <robot xmlns:xacro="http://ros.org/wiki/xacro">
-  <xacro:macro name="g1_29dof_lock_waist_rev_1_0" params="prefix">
+  <xacro:macro name="g1_29dof_rev_1_0" params="prefix">
   <material name="dark">
     <color rgba="0.2 0.2 0.2 1"/>
@@ -8,11 +8,11 @@
   </material>
   <mujoco>
-    <compiler meshdir="../meshes" discardvisual="false"/>
+    <compiler meshdir="meshes" discardvisual="false"/>
   </mujoco>
   <!-- [CAUTION] uncomment when convert to mujoco -->
   <!-- <link name="${prefix}world"></link>
-  <joint name="${prefix}floating_base_joint" type="floating">
-    <parent link="${prefix}world"/>
-    <child link="${prefix}pelvis"/>
+  <joint name="floating_base_joint" type="floating">
+    <parent link="world"/>
+    <child link="pelvis"/>
   </joint> -->
   <link name="${prefix}pelvis">
@@ -25,5 +25,5 @@
       <origin xyz="0 0 0" rpy="0 0 0"/>
       <geometry>
-        <mesh filename="package://g1_description/meshes/pelvis.STL"/>
+        <mesh filename="meshes/pelvis.STL"/>
       </geometry>
       <material name="dark"/>
@@ -39,18 +39,18 @@
       <origin xyz="0 0 0" rpy="0 0 0"/>
       <geometry>
-        <mesh filename="package://g1_description/meshes/pelvis_contour_link.STL"/>
-      </geometry>
-      <material name="white"/>
-    </visual>
-    <collision>
-      <origin xyz="0 0 0" rpy="0 0 0"/>
-      <geometry>
-        <mesh filename="package://g1_description/meshes/pelvis_contour_link.STL"/>
-      </geometry>
-    </collision>
-  </link>
-  <joint name="${prefix}pelvis_contour_joint" type="fixed">
-    <parent link="${prefix}pelvis"/>
-    <child link="${prefix}pelvis_contour_link"/>
+        <mesh filename="meshes/pelvis_contour_link.STL"/>
+      </geometry>
+      <material name="white"/>
+    </visual>
+    <collision>
+      <origin xyz="0 0 0" rpy="0 0 0"/>
+      <geometry>
+        <mesh filename="meshes/pelvis_contour_link.STL"/>
+      </geometry>
+    </collision>
+  </link>
+  <joint name="pelvis_contour_joint" type="fixed">
+    <parent link="pelvis"/>
+    <child link="pelvis_contour_link"/>
   </joint>
   <!-- Legs -->
@@ -64,5 +64,5 @@
       <origin xyz="0 0 0" rpy="0 0 0"/>
       <geometry>
-        <mesh filename="package://g1_description/meshes/left_hip_pitch_link.STL"/>
+        <mesh filename="meshes/left_hip_pitch_link.STL"/>
       </geometry>
       <material name="dark"/>
@@ -71,12 +71,12 @@
       <origin xyz="0 0 0" rpy="0 0 0"/>
       <geometry>
-        <mesh filename="package://g1_description/meshes/left_hip_pitch_link.STL"/>
-      </geometry>
-    </collision>
-  </link>
-  <joint name="${prefix}left_hip_pitch_joint" type="revolute">
+        <mesh filename="meshes/left_hip_pitch_link.STL"/>
+      </geometry>
+    </collision>
+  </link>
+  <joint name="left_hip_pitch_joint" type="revolute">
     <origin xyz="0 0.064452 -0.1027" rpy="0 0 0"/>
-    <parent link="${prefix}pelvis"/>
-    <child link="${prefix}left_hip_pitch_link"/>
+    <parent link="pelvis"/>
+    <child link="left_hip_pitch_link"/>
     <axis xyz="0 1 0"/>
     <limit lower="-2.5307" upper="2.8798" effort="88" velocity="32"/>
@@ -91,19 +91,19 @@
       <origin xyz="0 0 0" rpy="0 0 0"/>
       <geometry>
-        <mesh filename="package://g1_description/meshes/left_hip_roll_link.STL"/>
-      </geometry>
-      <material name="white"/>
-    </visual>
-    <collision>
-      <origin xyz="0 0 0" rpy="0 0 0"/>
-      <geometry>
-        <mesh filename="package://g1_description/meshes/left_hip_roll_link.STL"/>
-      </geometry>
-    </collision>
-  </link>
-  <joint name="${prefix}left_hip_roll_joint" type="revolute">
+        <mesh filename="meshes/left_hip_roll_link.STL"/>
+      </geometry>
+      <material name="white"/>
+    </visual>
+    <collision>
+      <origin xyz="0 0 0" rpy="0 0 0"/>
+      <geometry>
+        <mesh filename="meshes/left_hip_roll_link.STL"/>
+      </geometry>
+    </collision>
+  </link>
+  <joint name="left_hip_roll_joint" type="revolute">
     <origin xyz="0 0.052 -0.030465" rpy="0 -0.1749 0"/>
-    <parent link="${prefix}left_hip_pitch_link"/>
-    <child link="${prefix}left_hip_roll_link"/>
+    <parent link="left_hip_pitch_link"/>
+    <child link="left_hip_roll_link"/>
     <axis xyz="1 0 0"/>
     <limit lower="-0.5236" upper="2.9671" effort="139" velocity="20"/>
@@ -118,19 +118,19 @@
       <origin xyz="0 0 0" rpy="0 0 0"/>
       <geometry>
-        <mesh filename="package://g1_description/meshes/left_hip_yaw_link.STL"/>
-      </geometry>
-      <material name="white"/>
-    </visual>
-    <collision>
-      <origin xyz="0 0 0" rpy="0 0 0"/>
-      <geometry>
-        <mesh filename="package://g1_description/meshes/left_hip_yaw_link.STL"/>
-      </geometry>
-    </collision>
-  </link>
-  <joint name="${prefix}left_hip_yaw_joint" type="revolute">
+        <mesh filename="meshes/left_hip_yaw_link.STL"/>
+      </geometry>
+      <material name="white"/>
+    </visual>
+    <collision>
+      <origin xyz="0 0 0" rpy="0 0 0"/>
+      <geometry>
+        <mesh filename="meshes/left_hip_yaw_link.STL"/>
+      </geometry>
+    </collision>
+  </link>
+  <joint name="left_hip_yaw_joint" type="revolute">
     <origin xyz="0.025001 0 -0.12412" rpy="0 0 0"/>
-    <parent link="${prefix}left_hip_roll_link"/>
-    <child link="${prefix}left_hip_yaw_link"/>
+    <parent link="left_hip_roll_link"/>
+    <child link="left_hip_yaw_link"/>
     <axis xyz="0 0 1"/>
     <limit lower="-2.7576" upper="2.7576" effort="88" velocity="32"/>
@@ -145,19 +145,19 @@
       <origin xyz="0 0 0" rpy="0 0 0"/>
       <geometry>
-        <mesh filename="package://g1_description/meshes/left_knee_link.STL"/>
-      </geometry>
-      <material name="white"/>
-    </visual>
-    <collision>
-      <origin xyz="0 0 0" rpy="0 0 0"/>
-      <geometry>
-        <mesh filename="package://g1_description/meshes/left_knee_link.STL"/>
-      </geometry>
-    </collision>
-  </link>
-  <joint name="${prefix}left_knee_joint" type="revolute">
+        <mesh filename="meshes/left_knee_link.STL"/>
+      </geometry>
+      <material name="white"/>
+    </visual>
+    <collision>
+      <origin xyz="0 0 0" rpy="0 0 0"/>
+      <geometry>
+        <mesh filename="meshes/left_knee_link.STL"/>
+      </geometry>
+    </collision>
+  </link>
+  <joint name="left_knee_joint" type="revolute">
     <origin xyz="-0.078273 0.0021489 -0.17734" rpy="0 0.1749 0"/>
-    <parent link="${prefix}left_hip_yaw_link"/>
-    <child link="${prefix}left_knee_link"/>
+    <parent link="left_hip_yaw_link"/>
+    <child link="left_knee_link"/>
     <axis xyz="0 1 0"/>
     <limit lower="-0.087267" upper="2.8798" effort="139" velocity="20"/>
@@ -172,19 +172,19 @@
       <origin xyz="0 0 0" rpy="0 0 0"/>
       <geometry>
-        <mesh filename="package://g1_description/meshes/left_ankle_pitch_link.STL"/>
-      </geometry>
-      <material name="white"/>
-    </visual>
-    <collision>
-      <origin xyz="0 0 0" rpy="0 0 0"/>
-      <geometry>
-        <mesh filename="package://g1_description/meshes/left_ankle_pitch_link.STL"/>
-      </geometry>
-    </collision>
-  </link>
-  <joint name="${prefix}left_ankle_pitch_joint" type="revolute">
+        <mesh filename="meshes/left_ankle_pitch_link.STL"/>
+      </geometry>
+      <material name="white"/>
+    </visual>
+    <collision>
+      <origin xyz="0 0 0" rpy="0 0 0"/>
+      <geometry>
+        <mesh filename="meshes/left_ankle_pitch_link.STL"/>
+      </geometry>
+    </collision>
+  </link>
+  <joint name="left_ankle_pitch_joint" type="revolute">
     <origin xyz="0 -9.4445E-05 -0.30001" rpy="0 0 0"/>
-    <parent link="${prefix}left_knee_link"/>
-    <child link="${prefix}left_ankle_pitch_link"/>
+    <parent link="left_knee_link"/>
+    <child link="left_ankle_pitch_link"/>
     <axis xyz="0 1 0"/>
     <limit lower="-0.87267" upper="0.5236" effort="35" velocity="30"/>
@@ -199,5 +199,5 @@
       <origin xyz="0 0 0" rpy="0 0 0"/>
       <geometry>
-        <mesh filename="package://g1_description/meshes/left_ankle_roll_link.STL"/>
+        <mesh filename="meshes/left_ankle_roll_link.STL"/>
       </geometry>
       <material name="dark"/>
@@ -228,8 +228,8 @@
     </collision>
   </link>
-  <joint name="${prefix}left_ankle_roll_joint" type="revolute">
+  <joint name="left_ankle_roll_joint" type="revolute">
     <origin xyz="0 0 -0.017558" rpy="0 0 0"/>
-    <parent link="${prefix}left_ankle_pitch_link"/>
-    <child link="${prefix}left_ankle_roll_link"/>
+    <parent link="left_ankle_pitch_link"/>
+    <child link="left_ankle_roll_link"/>
     <axis xyz="1 0 0"/>
     <limit lower="-0.2618" upper="0.2618" effort="35" velocity="30"/>
@@ -244,5 +244,5 @@
       <origin xyz="0 0 0" rpy="0 0 0"/>
       <geometry>
-        <mesh filename="package://g1_description/meshes/right_hip_pitch_link.STL"/>
+        <mesh filename="meshes/right_hip_pitch_link.STL"/>
       </geometry>
       <material name="dark"/>
@@ -251,12 +251,12 @@
       <origin xyz="0 0 0" rpy="0 0 0"/>
       <geometry>
-        <mesh filename="package://g1_description/meshes/right_hip_pitch_link.STL"/>
-      </geometry>
-    </collision>
-  </link>
-  <joint name="${prefix}right_hip_pitch_joint" type="revolute">
+        <mesh filename="meshes/right_hip_pitch_link.STL"/>
+      </geometry>
+    </collision>
+  </link>
+  <joint name="right_hip_pitch_joint" type="revolute">
     <origin xyz="0 -0.064452 -0.1027" rpy="0 0 0"/>
-    <parent link="${prefix}pelvis"/>
-    <child link="${prefix}right_hip_pitch_link"/>
+    <parent link="pelvis"/>
+    <child link="right_hip_pitch_link"/>
     <axis xyz="0 1 0"/>
     <limit lower="-2.5307" upper="2.8798" effort="88" velocity="32"/>
@@ -271,19 +271,19 @@
       <origin xyz="0 0 0" rpy="0 0 0"/>
       <geometry>
-        <mesh filename="package://g1_description/meshes/right_hip_roll_link.STL"/>
-      </geometry>
-      <material name="white"/>
-    </visual>
-    <collision>
-      <origin xyz="0 0 0" rpy="0 0 0"/>
-      <geometry>
-        <mesh filename="package://g1_description/meshes/right_hip_roll_link.STL"/>
-      </geometry>
-    </collision>
-  </link>
-  <joint name="${prefix}right_hip_roll_joint" type="revolute">
+        <mesh filename="meshes/right_hip_roll_link.STL"/>
+      </geometry>
+      <material name="white"/>
+    </visual>
+    <collision>
+      <origin xyz="0 0 0" rpy="0 0 0"/>
+      <geometry>
+        <mesh filename="meshes/right_hip_roll_link.STL"/>
+      </geometry>
+    </collision>
+  </link>
+  <joint name="right_hip_roll_joint" type="revolute">
     <origin xyz="0 -0.052 -0.030465" rpy="0 -0.1749 0"/>
-    <parent link="${prefix}right_hip_pitch_link"/>
-    <child link="${prefix}right_hip_roll_link"/>
+    <parent link="right_hip_pitch_link"/>
+    <child link="right_hip_roll_link"/>
     <axis xyz="1 0 0"/>
     <limit lower="-2.9671" upper="0.5236" effort="139" velocity="20"/>
@@ -298,19 +298,19 @@
       <origin xyz="0 0 0" rpy="0 0 0"/>
       <geometry>
-        <mesh filename="package://g1_description/meshes/right_hip_yaw_link.STL"/>
-      </geometry>
-      <material name="white"/>
-    </visual>
-    <collision>
-      <origin xyz="0 0 0" rpy="0 0 0"/>
-      <geometry>
-        <mesh filename="package://g1_description/meshes/right_hip_yaw_link.STL"/>
-      </geometry>
-    </collision>
-  </link>
-  <joint name="${prefix}right_hip_yaw_joint" type="revolute">
+        <mesh filename="meshes/right_hip_yaw_link.STL"/>
+      </geometry>
+      <material name="white"/>
+    </visual>
+    <collision>
+      <origin xyz="0 0 0" rpy="0 0 0"/>
+      <geometry>
+        <mesh filename="meshes/right_hip_yaw_link.STL"/>
+      </geometry>
+    </collision>
+  </link>
+  <joint name="right_hip_yaw_joint" type="revolute">
     <origin xyz="0.025001 0 -0.12412" rpy="0 0 0"/>
-    <parent link="${prefix}right_hip_roll_link"/>
-    <child link="${prefix}right_hip_yaw_link"/>
+    <parent link="right_hip_roll_link"/>
+    <child link="right_hip_yaw_link"/>
     <axis xyz="0 0 1"/>
     <limit lower="-2.7576" upper="2.7576" effort="88" velocity="32"/>
@@ -325,19 +325,19 @@
       <origin xyz="0 0 0" rpy="0 0 0"/>
       <geometry>
-        <mesh filename="package://g1_description/meshes/right_knee_link.STL"/>
-      </geometry>
-      <material name="white"/>
-    </visual>
-    <collision>
-      <origin xyz="0 0 0" rpy="0 0 0"/>
-      <geometry>
-        <mesh filename="package://g1_description/meshes/right_knee_link.STL"/>
-      </geometry>
-    </collision>
-  </link>
-  <joint name="${prefix}right_knee_joint" type="revolute">
+        <mesh filename="meshes/right_knee_link.STL"/>
+      </geometry>
+      <material name="white"/>
+    </visual>
+    <collision>
+      <origin xyz="0 0 0" rpy="0 0 0"/>
+      <geometry>
+        <mesh filename="meshes/right_knee_link.STL"/>
+      </geometry>
+    </collision>
+  </link>
+  <joint name="right_knee_joint" type="revolute">
     <origin xyz="-0.078273 -0.0021489 -0.17734" rpy="0 0.1749 0"/>
-    <parent link="${prefix}right_hip_yaw_link"/>
-    <child link="${prefix}right_knee_link"/>
+    <parent link="right_hip_yaw_link"/>
+    <child link="right_knee_link"/>
     <axis xyz="0 1 0"/>
     <limit lower="-0.087267" upper="2.8798" effort="139" velocity="20"/>
@@ -352,19 +352,19 @@
       <origin xyz="0 0 0" rpy="0 0 0"/>
       <geometry>
-        <mesh filename="package://g1_description/meshes/right_ankle_pitch_link.STL"/>
-      </geometry>
-      <material name="white"/>
-    </visual>
-    <collision>
-      <origin xyz="0 0 0" rpy="0 0 0"/>
-      <geometry>
-        <mesh filename="package://g1_description/meshes/right_ankle_pitch_link.STL"/>
-      </geometry>
-    </collision>
-  </link>
-  <joint name="${prefix}right_ankle_pitch_joint" type="revolute">
+        <mesh filename="meshes/right_ankle_pitch_link.STL"/>
+      </geometry>
+      <material name="white"/>
+    </visual>
+    <collision>
+      <origin xyz="0 0 0" rpy="0 0 0"/>
+      <geometry>
+        <mesh filename="meshes/right_ankle_pitch_link.STL"/>
+      </geometry>
+    </collision>
+  </link>
+  <joint name="right_ankle_pitch_joint" type="revolute">
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