Commit message: Reconstruct the project

File: legged_robot_description/go2_description/urdf/leg.xacro (robot description, xacro)
@@ -1,5 +1,5 @@
 <?xml version="1.0"?>
 <robot xmlns:xacro="http://www.ros.org/wiki/xacro">
-    <xacro:include filename="$(find go2_description)/xacro/transmission.xacro"/>
+    <xacro:include filename="$(find go2_description)/urdf/transmission.xacro"/>
     <xacro:macro name="leg" params="name mirror mirror_dae front_hind front_hind_dae">
         <joint name="${name}_hip_joint" type="revolute">

File: legged_robot_description/go2_description/urdf/robot.xacro (robot description, xacro)
@@ -4,12 +4,12 @@
     <xacro:arg name="prefix" default="" />
     <xacro:arg name="enable_sim" default="true" />
-    <xacro:arg name="network_interface" default="lo" />
-    <xacro:include filename="$(find go2_description)/xacro/const.xacro"/>
-    <xacro:include filename="$(find go2_description)/xacro/materials.xacro"/>
-    <xacro:include filename="$(find go2_description)/xacro/leg.xacro"/>
-    <!-- <xacro:include filename="$(find go2_description)/xacro/stairs.xacro"/> -->
-    <xacro:include filename="$(find go2_description)/xacro/gazebo.xacro"/>
+    <xacro:arg name="enable_lowlevel_write" default="true" />
+    <xacro:include filename="$(find go2_description)/urdf/const.xacro"/>
+    <xacro:include filename="$(find go2_description)/urdf/materials.xacro"/>
+    <xacro:include filename="$(find go2_description)/urdf/leg.xacro"/>
+    <!-- <xacro:include filename="$(find go2_description)/urdf/stairs.xacro"/> -->
+    <xacro:include filename="$(find go2_description)/urdf/gazebo.xacro"/>
     <!-- <xacro:include filename="$(find go2_gazebo)/launch/stairs.urdf.xacro"/> -->
-    <xacro:include filename="$(find go2_description)/xacro/ros2_control.xacro"/>
+    <xacro:include filename="$(find go2_description)/urdf/ros2_control.xacro"/>
     <!-- <xacro:stairs stairs="15" xpos="0" ypos="0" zpos="0" /> -->
     <!-- Rotor related joint and link is only for demonstrate location. -->
@@ -85,4 +85,11 @@
         </collision>
     </link>
+    <joint name="utlidar_joint" type="fixed">
+        <origin xyz="0.28945 0 -0.046825" rpy="0 2.8782 0" />
+        <parent link="trunk" />
+        <child link="utlidar_link" />
+    </joint>
+    <link name="utlidar_link">
+    </link>
     <joint name="front_camera_joint" type="fixed">
         <parent link="trunk"/>
@@ -125,4 +132,4 @@
         prefix="$(arg prefix)"
         enable_sim="$(arg enable_sim)"
-        network_interface="$(arg network_interface)"/>
+        enable_lowlevel_write="$(arg enable_lowlevel_write)"/>
 </robot>

File: legged_robot_description/go2_description/urdf/ros2_control.xacro (robot description, xacro)
@@ -1,5 +1,5 @@
 <?xml version="1.0"?>
 <robot xmlns:xacro="http://www.ros.org/wiki/xacro">
-  <xacro:macro name="go2_ros2_control" params="prefix enable_sim:=false network_interface:=lo">
+  <xacro:macro name="go2_ros2_control" params="prefix enable_sim:=false enable_lowlevel_write:=true">
     <ros2_control name="go2_ros2_control" type="system">
       <xacro:if value="${enable_sim}">
@@ -11,5 +11,5 @@
         <hardware>
           <plugin>legged_ros2_control/Go2SystemInterface</plugin>
-          <param name="network_interface">${network_interface}</param>
+          <param name="enable_lowlevel_write">${enable_lowlevel_write}</param>
         </hardware>
       </xacro:unless>

File: legged_robot_description/go2_description/urdf/test.urdf (robot description, URDF)
Before this commit: robot go2, 32 links, 31 joints
Links:
- added link utlidar_link, mass 0
- link trunk: geometry collision box size=0.3762 0.0935 0.114; visual mesh filename=package://go2_description/meshes/base.dae scale=1 1 1
Joints:
- added joint utlidar_joint: type fixed, parent trunk, child utlidar_link, origin xyz=0.28945 0 -0.046825 rpy=0 2.8782 0, axis 0 0 0
